Commit message: Correccion en el Xacro (valor en radianes)

File: src/mi_robot_mecanum/urdf/mi_robot.urdf.xacro (robot description, xacro)
@@ -86,15 +86,15 @@
     <visual>
       <origin xyz="0 0 0" rpy="0 0 0"/>
-      <geometry><cylinder radius="0.0515" length="0.041"/></geometry>
+      <geometry><cylinder radius="0.038" length="0.041"/></geometry>
       <material name="gris"><color rgba="0.7 0.7 0.7 1"/></material>
     </visual>
     <collision>
       <origin xyz="0 0 0" rpy="0 0 0"/>
-      <geometry><cylinder radius="0.0515" length="0.041"/></geometry>
+      <geometry><cylinder radius="0.038" length="0.041"/></geometry>
     </collision>
     <inertial>
       <origin xyz="0 0 0" rpy="0 0 0"/>
       <mass value="0.19"/>
-      <xacro:inercia_cilindro m="0.19" r="0.0515" h="0.041"/>
+      <xacro:inercia_cilindro m="0.19" r="0.038" h="0.041"/>
     </inertial>
   </link>
@@ -109,5 +109,5 @@
       <topic>/scan</topic>
       <gz_frame_id>lidar_link</gz_frame_id>
-      <update_rate>10</update_rate>
+      <update_rate>8</update_rate>
       <always_on>1</always_on>
       <visualize>true</visualize>
@@ -115,5 +115,5 @@
         <scan>
           <horizontal>
-            <samples>360</samples>          <!-- muestras por vuelta -->
+            <samples>2000</samples>          <!-- muestras por vuelta -->
             <resolution>1</resolution>
             <min_angle>-3.14159</min_angle>
@@ -122,6 +122,6 @@
         </scan>
         <range>
-          <min>0.12</min>
-          <max>12.0</max>
+          <min>0.2</min>
+          <max>25.0</max>
           <resolution>0.01</resolution>
         </range>
@@ -168,9 +168,9 @@
     <sensor name="astra" type="rgbd_camera">
       <topic>/camara</topic>
-      <gz_frame_id>camara_optica_link</gz_frame_id>
+      <gz_frame_id>camara_link</gz_frame_id>
       <update_rate>30</update_rate>
       <always_on>1</always_on>
       <camera>
-        <horizontal_fov>1.10130276</horizontal_fov>   <!-- 63.1 grados, en radianes -->
+        <horizontal_fov>1.0193</horizontal_fov>   <!-- en radianes -->
         <image>
           <width>640</width>
